Commit message: remove grippers

File: kuka_kr60/kuka_kr60_support/urdf/UM_KR60_setup.urdf (robot description, URDF)
Before this commit: robot UM_KR60_setup, 19 links, 18 joints
Links:
- removed link left_gripper
- removed link right_gripper
Joints:
- removed joint left_tool0-gripper
- removed joint right_tool0-gripper

File: kuka_kr60/kuka_kr60_support/urdf/UM_KR60_setup.xacro (robot description, xacro)
@@ -2,7 +2,19 @@
 <!--Generates a urdf from the macro in kr120r2500pro_macro.xacro -->
 <robot name="UM_KR60_setup" xmlns:xacro="http://wiki.ros.org/xacro">
+    <xacro:property name="left_prefix" value="left_" />
+    <xacro:property name="right_prefix" value="right_" />
     <xacro:include filename="$(find kuka_kr60_support)/urdf/kr60_macro.xacro" />
     <link name="world"/>
-    <xacro:kuka_kr60 prefix="left_" link_to="world" xyz_offset="0.0 -2.390051 0.0"/>
-    <xacro:kuka_kr60 prefix="right_" link_to="world" xyz_offset="0.0 0.0 0.0"/>
+    <joint name="${left_prefix}grounding" type="fixed">
+        <parent link="world"/>
+	<child link="${left_prefix}base_link"/>
+	<origin xyz="0.0 -2.390051 0.0" rpy="0.0 0.0 0.0"/>
+    </joint>
+    <joint name="${right_prefix}grounding" type="fixed">
+        <parent link="world"/>
+	<child link="${right_prefix}base_link"/>
+	<origin xyz="0.0 0.0 0.0" rpy="0.0 0.0 0.0"/>
+    </joint>
+    <xacro:kuka_kr60 prefix="${left_prefix}"/>
+    <xacro:kuka_kr60 prefix="${right_prefix}"/>
 </robot>

File: kuka_kr60/kuka_kr60_support/urdf/kr60_macro.xacro (robot description, xacro)
@@ -2,5 +2,5 @@
 <robot xmlns:xacro="http://wiki.ros.org/xacro">
   <xacro:property name="DEG2RAD" value="0.017453292519943295"/>
-  <xacro:macro name="kuka_kr60" params="prefix link_to xyz_offset">
+  <xacro:macro name="kuka_kr60" params="prefix">
 		<xacro:macro name="transmission_block" params="joint_name">
 			<transmission name="tran1">
@@ -170,42 +170,4 @@
  <!-- tool 0 -->
     <!-- This frame corresponds to the $FLANGE coordinate system in KUKA KRC controllers. -->
-		<!--OCIMA Gripper-->
-		<link name="${prefix}gripper">
-      <inertial>
-      <origin
-        xyz="-0.0428764766835783 -0.013530986668562 -0.0481091446071806"
-        rpy="0 0 0" />
-      <mass
-        value="4.45066934712782" />
-      <inertia
-        ixx="0.0280534429483876"
-        ixy="0.00203411158636486"
-        ixz="-0.00280489820899368"
-        iyy="0.12704521558317"
-        iyz="-0.000926853755642866"
-        izz="0.107306139125527" />
-    </inertial>
-    <visual>
-      <origin
-        xyz="0 0 0"
-        rpy="0 0 0" />
-      <geometry>
-			<mesh
-          filename="package://gripper_ocima/meshes/base_link.dae" />
-		  </geometry>
-			<material name="Orange" >
-       <!--<color rgba="1 0.49 0.31 1" />-->
-      </material>
-    </visual>
-    <collision>
-      <origin
-        xyz="0 0 0"
-        rpy="0 0 0" />
-      <geometry>
-        <mesh
-          filename="package://gripper_ocima/meshes/base_link.STL" />
-  </geometry>
-    </collision>
-    </link>
     <!-- END LINKS -->
     <!-- JOINTS -->
@@ -274,17 +236,6 @@
 			<hardwareInterface>hardware_interface/PositionJointInterface</hardwareInterface>
     </joint>
-<!-- gripper frame - fixed frame -->
-    <joint name="${prefix}tool0-gripper" type="fixed">
-      <parent link="${prefix}tool0"/>
-      <child link="${prefix}gripper"/>
-			<origin xyz="0.41 -0.33 -0.02" rpy="-${DEG2RAD*90} 0 ${DEG2RAD*90}"/>
-    </joint>
     <!-- END JOINTS -->
     <!-- ROS base_link to KUKA $ROBROOT coordinate system transform  -->
-		<joint name="${prefix}grounding" type="fixed">
-			<parent link="${link_to}"/>
-			<child link="${prefix}base_link"/>
-			<origin xyz="${xyz_offset}" rpy="0.0 0.0 0.0"/>
-		</joint>
 		<xacro:transmission_block joint_name="${prefix}joint_a1"/>
 		<xacro:transmission_block joint_name="${prefix}joint_a2"/>

Commit message: changing tool0 offset

File: kuka_kr60/kuka_kr60_support/urdf/UM_KR60_setup.urdf (robot description, URDF)
Before this commit: robot UM_KR60_setup, 17 links, 16 joints
Joints:
- joint left_joint_a6-tool0: origin xyz=0.215 0 0 rpy=0 1.57079632679 0 -> xyz=0.038 0 0 rpy=0 1.57079632679 0
- joint right_joint_a6-tool0: origin xyz=0.215 0 0 rpy=0 1.57079632679 0 -> xyz=0.038 0 0 rpy=0 1.57079632679 0

File: kuka_kr60/kuka_kr60_support/urdf/kr60_macro.xacro (robot description, xacro)
@@ -233,5 +233,5 @@
       <parent link="${prefix}link_6"/>
       <child link="${prefix}tool0"/>
-      <origin xyz="0.215 0 0" rpy="0 ${DEG2RAD * 90} 0"/>
+      <origin xyz="0.038 0 0" rpy="0 ${DEG2RAD * 90} 0"/>
 			<hardwareInterface>hardware_interface/PositionJointInterface</hardwareInterface>
     </joint>
